File: elec_angle_sensor/elec_angle_sensor.kicad_pcb (KiCad board)
At the start: 4 copper layers, 0 parts

Commit message: [update] Full schematic + positionning
Parts:
- added C25: 100n, Capacitor_SMD:C_0402_1005Metric, F.Cu at (130.7, 54.6)
- added D1: SP0503BAHT, Package_TO_SOT_SMD:SOT-143, F.Cu at (129.4, 49.5)
- added FID1: DNP Fiducial, Fiducial:Fiducial_1mm_Mask2mm, F.Cu at (129.6, 42.6)
- added FID2: DNP Fiducial, Fiducial:Fiducial_1mm_Mask2mm, F.Cu at (130.4, 57.8)
- added FID3: DNP Fiducial, Fiducial:Fiducial_1mm_Mask2mm, F.Cu at (123.3, 55.0)
- added G1: qwiic_Logo, Library_Pollen:Logo_qwiic_5mm, F.Cu at (110.4, 41.4)
- added H2: Logo HF 2025, Library_Pollen:Logo_HF_2025, F.Cu at (112.8, 44.4)
- added H3: DNP Logo Pollen 2021, Library_Pollen:Logo_Pollen_2021_sq, F.Cu at (105.0, 43.2)
- added H4: Mounting Holes M2,5, MountingHole:MountingHole_2.7mm_M2.5_ISO7380_Pad_TopBottom, F.Cu at (124.4, 42.6)
- added H5: MountingHole_Pad, MountingHole:MountingHole_2.7mm_M2.5_ISO7380_Pad_TopBottom, F.Cu at (134.4, 57.6)
- added H6: Centering Hole 2 mm, Library_Pollen:MountingHole_2.0mm, F.Cu at (124.4, 57.6)
- added H7: Centering Hole 2 mm, Library_Pollen:MountingHole_2.0mm, F.Cu at (134.4, 42.6)
- added J1: JST SH, Connector_JST:JST_SH_SM04B-SRSS-TB_1x04-1MP_P1.00mm_Horizontal, F.Cu at (134.4, 49.7)
- added J7: JST SH, Connector_JST:JST_SH_SM04B-SRSS-TB_1x04-1MP_P1.00mm_Horizontal, F.Cu at (124.4, 49.6)
- added R1: DNP-10k, Resistor_SMD:R_0402_1005Metric, F.Cu at (126.7, 54.5)
- added R2: DNP-10k, Resistor_SMD:R_0402_1005Metric, F.Cu at (128.7, 54.5)
- added U1: AS5600L, Package_SO:SOIC-8_3.9x4.9mm_P1.27mm, B.Cu at (128.3, 49.6)
Other:
- board outline added: 17 x 21 mm
- board text added: "!! Prévoir une place pour marquer l'adresse I2C du capteur d'angle"
