File: elec_angle_sensor/elec_angle_sensor.kicad_sch (KiCad schematic)
At the start: 19 parts, among them J1 JST SH, J7 JST SH, U1 AS5600L

Commit message: [added] Production files
Other:
- note added: "12/03/2026"
- note removed: "dd/mm/2026"
