File: elec_gripette_hub_and_dyn/elec_gripette_hub_and_dyn.kicad_pcb (KiCad board)
At the start: 4 copper layers, 65 x 30 mm, 95 parts, among them J1 pico4, J2 JST EH 2, J3 Pogo-pin, J4 Dynamixel-3, J5 Dynamixel-3, J6 Pogo-pin, J7 Pogo-pin 2A, J8 Pogo-pin 2A, J9 Dynamixel-3, Q1 MMBT3906, Q2 SI2312CDS-T1-GE3, U1 FE1.1s_24-Pin_WQFN, U2 24C02S, U3 CH343P, U4 SN74LVC1G125DBV, U5 SN74LVC1G126DBVR, U6 MP2338, U7 AP63205, U8 LM5050-1, Y1 12MHz

Commit message: [update] SCH B1-RC1
Parts:
- added C22: 100n, Capacitor_SMD:C_0603_1608Metric, F.Cu at (137.7, 73.0)
- added C23: 100n, Capacitor_SMD:C_0603_1608Metric, F.Cu at (157.8, 44.8)
- added C24: 100n, Capacitor_SMD:C_0603_1608Metric, F.Cu at (157.8, 47.3)
- added D10: D_Schottky 3A, Diode_SMD:D_SMA, F.Cu at (81.4, 18.0)
- added D12: 5V1, Diode_SMD:D_SOD-323, F.Cu at (152.9, 54.2)
- added J10: Pogo-pin 2A, LCSC_parts_lib:CONN-TH_YZ08415060P-02_pogo, B.Cu at (87.6, 32.7)
- added J13: Pogo-pin 2A, LCSC_parts_lib:CONN-TH_YZ08415060P-02_pogo, B.Cu at (99.4, 41.9)
- added J14: Pogo-pin 2A, LCSC_parts_lib:CONN-TH_YZ08415060P-02_pogo, B.Cu at (102.9, 41.9)
- added Q3: MMBT3906, Package_TO_SOT_SMD:SOT-23, F.Cu at (138.2, 63.3)
- added R17: 0R, Resistor_SMD:R_0402_1005Metric, F.Cu at (126.5, 52.1)
- added R29: 0R, Resistor_SMD:R_0402_1005Metric, F.Cu at (126.5, 54.0)
- added R30: DNP, Resistor_SMD:R_0603_1608Metric, F.Cu at (78.9, 27.9)
- added R31: DNP, Resistor_SMD:R_0603_1608Metric, F.Cu at (78.9, 30.4)
- added R32: 243k, Resistor_SMD:R_0402_1005Metric, F.Cu at (82.4, 29.6)
- added R33: 0R, Resistor_SMD:R_0402_1005Metric, F.Cu at (149.2, 44.5)
- added R34: 0R, Resistor_SMD:R_0402_1005Metric, F.Cu at (149.2, 46.5)
- added R35: 10k, Resistor_SMD:R_0402_1005Metric, F.Cu at (149.2, 48.5)
- added R36: 10k, Resistor_SMD:R_0402_1005Metric, F.Cu at (149.2, 50.5)
- added R37: 20k, Resistor_SMD:R_0402_1005Metric, F.Cu at (149.2, 52.5)
- added R38: 10k, Resistor_SMD:R_0402_1005Metric, F.Cu at (149.2, 54.5)
- added R39: 10k, Resistor_SMD:R_0402_1005Metric, F.Cu at (149.2, 56.5)
- added R40: 150R, Resistor_SMD:R_0402_1005Metric, F.Cu at (149.2, 58.4)
- added TH2: 100R thermistor, Resistor_SMD:R_0603_1608Metric, F.Cu at (157.8, 49.8)
- added U10: SN74LVC1G126DBVR, Package_TO_SOT_SMD:SOT-23-5, F.Cu at (153.3, 50.5)
- added U9: TPS54560BDDA, Package_SO:Texas_R-PDSO-G8_EP2.95x4.9mm_Mask2.4x3.1mm_ThermalVias, F.Cu at (81.2, 23.4)
- C12: value 22n -> 4n7
- C19: value 100p 50V -> 47p
- J3, J6: value Pogo-pin -> Pogo-pin 4mm
- J7: value Pogo-pin 2A -> Pogo-pin 2A 4mm
- R18: value 10k -> 16k9
- R19: value DNP - 0R -> DNP-0R
- R21: value 120k -> 62k
- R22: value 9k1 -> 8k2
- R23: value 160k -> DNP - 0R
- R26: value 6k8 -> 7k5
- U6: value MP2338 -> SN74LVC1G125DBV; footprint LCSC_parts_lib:SOT-583-8_L2.1-W1.2-P0.50-LS1.6-BR -> Package_TO_SOT_SMD:SOT-23-5
- moved U6 75.8 mm to (153.3, 45.9)
- moved R23 55.9 mm to (141.2, 72.8), turned to 0 degrees
- moved C12 25.3 mm to (85.3, 27.6), turned to 0 degrees
- moved R18 24.6 mm to (82.4, 27.6), turned to 0 degrees
- moved C19 23.4 mm to (85.3, 29.6), turned to 0 degrees
- moved J8 6.52 mm to (71.7, 72.2)
- moved R16 3.35 mm to (76.0, 53.0)
- moved C14 2.06 mm to (77.3, 45.6)
- moved J3 1.00 mm to (76.9, 72.7)
- moved J6 1.00 mm to (79.1, 72.7)
Connections:
- net /Dynamixel 3/Dynamixel_dir renamed /Dynamixel-TTL over USB/Dynamixel_dir
- net /Dynamixel 3/USB_DynN renamed /Dynamixel-TTL over USB/USB_DynN
- net /Dynamixel 3/USB_DynP renamed /Dynamixel-TTL over USB/USB_DynP
- net Net-(D9-K) renamed /Dynamixel-TTL over USB/Dyn_data
- C12 pad 1: GND -> Net-(C12-Pad1)
- C12 pad 2: Net-(U6-SS) -> GND
- C14 pad 1: Net-(U6-SW) -> Net-(D10-K)
- C14 pad 2: Net-(U6-BST) -> Net-(U9-BOOT)
- C19 pad 1: Net-(C16-Pad1) -> Net-(U9-COMP)
- C19 pad 2: Net-(C19-Pad2) -> GND
- C9 pad 1: VBUS -> +BATT
- L2 pad 2: Net-(U6-SW) -> Net-(D10-K)
- R10 pad 1: /Dynamixel 3/Tx -> /Dynamixel-TTL over USB/Tx
- R11 pad 1: /Dynamixel 3/Tx -> /Dynamixel-TTL over USB/Tx
- R13 pad 2: /Dynamixel 3/Rx -> /Dynamixel-TTL over USB/Rx
- R16 pad 1: Net-(U6-PG) -> Net-(C16-Pad1)
- R16 pad 2: Net-(C16-Pad1) -> Net-(R16-Pad2)
- R18 pad 1: Net-(U6-FB) -> Net-(U9-COMP)
- R18 pad 2: Net-(C19-Pad2) -> Net-(C12-Pad1)
- R19 pad 1: Net-(C19-Pad2) -> Net-(U9-FB)
- R20 pad 1: Net-(C19-Pad2) -> Net-(U9-FB)
- R20 pad 2: Net-(R20-Pad2) -> Net-(R16-Pad2)
- R23 pad 1: Net-(R20-Pad2) -> Net-(U1-~{XRSTJ})
- R23 pad 2: Net-(C16-Pad1) -> Net-(J10-Pad1)
- R26 pad 2: Net-(R20-Pad2) -> Net-(R16-Pad2)
- U3 pad 4: /Dynamixel 3/Tx -> Net-(U3-TXD)
- U3 pad 5: /Dynamixel 3/Rx -> Net-(U3-RXD)
- U4 pad 4: /Dynamixel 3/Rx -> /Dynamixel-TTL over USB/Rx
- U5 pad 2: /Dynamixel 3/Tx -> /Dynamixel-TTL over USB/Tx
- U6 pad 1: Net-(U6-PG) -> /Dynamixel-TTL/Dynamixel_dir
- U6 pad 2: +BATT -> Net-(R39-Pad2)
- U6 pad 3: Net-(U6-SW) -> GND
- U6 pad 4: GND -> /Dynamixel-TTL/Rx
- U6 pad 5: Net-(U6-BST) -> +5V
- U7 pad 2: VBUS -> +BATT
- U7 pad 3: VBUS -> +BATT
Routing:
- net Net-(C19-Pad2): track 17.7 -> 0.00 mm, vias 2 -> 0
- net Net-(U3-TXD): track 0.00 -> 16.6 mm
- net /Dynamixel 3/Tx: track 16.6 -> 0.00 mm
- net Net-(U3-RXD): track 0.00 -> 14.0 mm
- net /Dynamixel 3/Rx: track 14.0 -> 0.00 mm
- net +BATT: track 27.0 -> 14.1 mm, vias 2 -> 0
- net Net-(U6-SW): track 10.6 -> 0.00 mm
- net /USB hub/rasp_D+: track 18.7 -> 11.0 mm
- net Net-(C16-Pad1): track 29.5 -> 24.6 mm
- net /USB hub/rasp_D-: track 16.7 -> 12.3 mm
- net Net-(U9-FB): track 0.00 -> 2.88 mm, vias 0 -> 1
- net Net-(R20-Pad2): track 2.52 -> 0.00 mm
- net Net-(R16-Pad2): track 0.00 -> 2.52 mm
- net GND: track 78.4 -> 75.9 mm, vias 32 -> 30
- net Net-(U6-BST): track 2.00 -> 0.00 mm
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Other:
- board text added: "ASE01201-B1"
- board text removed: "ASE01201-A1"

Commit message: [update] SCH + PCB B1-RC1
Parts:
- removed TP1: TestPoint, TestPoint:TestPoint_Pad_D1.0mm
- J10, J13, J14: value Pogo-pin 2A -> Pogo-pin 4mm; footprint LCSC_parts_lib:CONN-TH_YZ08415060P-02_pogo -> LCSC_parts_lib:CONN-TH_YZ95315064P-01_pogo
- J8: value Pogo-pin 2A -> Pogo-pin 2A 4mm
- R30, R31: footprint Resistor_SMD:R_0603_1608Metric -> Resistor_SMD:R_0402_1005Metric
- moved TH2 63.2 mm to (95.5, 60.2), turned to 180 degrees
- moved D12 55.1 mm to (98.0, 59.4), turned to 90 degrees
- moved C23 53.2 mm to (105.4, 53.4), turned to 90 degrees
- moved C22 52.8 mm to (84.9, 73.4)
- moved U6 52.4 mm to (101.5, 54.0)
- moved R40 49.7 mm to (99.5, 58.7), turned to -90 degrees
- moved R34 48.4 mm to (100.9, 48.9), turned to -90 degrees
- moved R23 47.9 mm to (98.3, 51.4), turned to 90 degrees
- moved C24 47.1 mm to (110.9, 51.1)
- moved R33 46.0 mm to (103.4, 48.9), turned to -90 degrees
- moved R38 45.1 mm to (104.2, 54.5), turned to -90 degrees
- moved R36 44.5 mm to (104.8, 48.9), turned to 90 degrees
- moved R35 44.0 mm to (105.3, 50.4)
- moved U10 43.0 mm to (110.4, 53.7)
- moved R37 40.4 mm to (109.2, 46.4), turned to -90 degrees
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Connections:
- net /Dynamixel-TTL over USB/USB_DynN renamed /Dynamixel-TTL over USB/hub_DP2-
- net /Dynamixel-TTL over USB/USB_DynP renamed /Dynamixel-TTL over USB/hub_DP2+
- net /USB hub/DM+ renamed /USB hub/hub_DU+
- net /USB hub/DM- renamed /USB hub/hub_DU-
- net /USB hub/hub_dp3N renamed /USB hub/hub_DP3-
- net /USB hub/hub_dp3P renamed /USB hub/hub_DP3+
- net /USB hub/hub_dp4N renamed /USB hub/hub_DP4-
- net /USB hub/hub_dp4P renamed /USB hub/hub_DP4+
- net /USB hub/rasp_D+ renamed /USB hub/hub_DP1+
- net /USB hub/rasp_D- renamed /USB hub/hub_DP1-
- U3 pad 12: Net-(U3-~{DTR}) -> unconnected-(U3-~{DTR}-Pad12)
Routing:
- net VBUS: track 48.8 -> 16.6 mm
- net Net-(U1-~{XRSTJ}): track 2.50 -> 27.4 mm, vias 0 -> 4
- net +BATT: track 14.1 -> 34.6 mm
- net Net-(R39-Pad2): track 0.00 -> 18.1 mm
- net /Dynamixel-TTL/Dynamixel_dir: track 0.00 -> 16.8 mm, vias 0 -> 2
- net /Dynamixel-TTL over USB/Tx: track 0.00 -> 15.0 mm
- net Net-(D10-K): track 0.00 -> 14.7 mm
- net /Dynamixel-TTL over USB/hub_DP2+: track 29.3 -> 16.2 mm
- net /Dynamixel-TTL over USB/hub_DP2-: track 28.5 -> 15.4 mm
- net Net-(D2-K): track 39.4 -> 29.9 mm
- net Net-(U1-LED1/EESCL): track 39.5 -> 30.2 mm
- net /Dynamixel-TTL/Tx: track 0.00 -> 8.82 mm
- net +5V: track 154.8 -> 163.2 mm, vias 8 -> 11
- net /USB hub/hub_DP4-: track 13.4 -> 5.59 mm
- net /Dynamixel-TTL/Rx: track 0.00 -> 7.78 mm
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Other:
- board text added: "1"
- board text added: "1,6 mm PCB thickness 35 um (1 oz) copper"
- board text added: "2"
- board text added: "3"
- board text added: "4"
- board text added: "Rst"
- board text added: "Rx"
- board text added: "Tx"
- board text removed: "1 mm PCB thickness 35 um (1 oz) copper"
- board text removed: "USB1"

Commit message: [update] Before review
Parts:
- R23, R24: value DNP - 0R -> DNP-0R; footprint Resistor_SMD:R_0402_1005Metric -> Resistor_SMD:R_0603_1608Metric
- moved FID2 29.9 mm to (117.4, 53.6)
- moved FID3 9.44 mm to (98.4, 46.6)
- moved D2 3.60 mm to (109.3, 71.7)
- moved D7 3.00 mm to (109.3, 70.1)
- moved FID1 2.04 mm to (63.4, 72.6)
- moved D6 1.90 mm to (109.3, 73.3)
- moved D4 1.30 mm to (109.3, 68.5)
- moved R4 0.80 mm to (111.7, 70.1)
- moved R5 0.56 mm to (111.7, 72.4)
- moved J1 0.55 mm to (74.7, 72.1)
- moved R23 0.50 mm to (98.3, 51.9)
- moved U8 0.41 mm to (68.9, 69.5)
- moved U4 0.30 mm to (113.8, 57.3)
- moved R24 0.10 mm to (114.9, 59.9)
Routing:
- net GND: track 74.1 -> 83.1 mm, vias 37 -> 43
- net Net-(D2-A): track 2.96 -> 6.36 mm
- net Net-(U1-LED1/EESCL): track 30.2 -> 33.4 mm
- net Net-(D6-A): track 3.13 -> 4.74 mm
- net Net-(U1-~{XRSTJ}): track 27.4 -> 26.7 mm
- net /USB hub/hub_DU+: track 13.1 -> 12.5 mm
- net Net-(J1-Pin_2): track 10.5 -> 10.00 mm
- net /USB hub/hub_DU-: track 13.1 -> 12.5 mm
