File: elec_gripette_hub_and_dyn/elec_gripette_hub_and_dyn.kicad_pcb (KiCad board)
At the start: 4 copper layers, 65 x 30 mm, 119 parts, among them J1 pico4, J10 Pogo-pin 4mm, J13 Pogo-pin 4mm, J14 Pogo-pin 4mm, J2 JST EH 2, J3 Pogo-pin 4mm, J4 Dynamixel-3, J5 Dynamixel-3, J6 Pogo-pin 4mm, J7 Pogo-pin 2A 4mm, J8 Pogo-pin 2A 4mm, J9 Dynamixel-3, Q1 MMBT3906, Q2 SI2312CDS-T1-GE3, Q3 MMBT3906, U1 FE1.1s_24-Pin_WQFN, U10 SN74LVC1G126DBVR, U2 24C02S, U3 CH343P, U4 SN74LVC1G125DBV, U5 SN74LVC1G126DBVR, U6 SN74LVC1G125DBV, U7 AP63205, U8 LM5050-1, U9 TPS54560BDDA, Y1 12MHz

Commit message: [update] review by Claude. Corrections, RC2
Parts:
- added C25: 1u, Capacitor_SMD:C_0603_1608Metric, F.Cu at (106.9, 55.8)
- added C26: 1u, Capacitor_SMD:C_0603_1608Metric, F.Cu at (104.3, 52.1)
- added C27: 3,3u 35V, Capacitor_SMD:C_0805_2012Metric, F.Cu at (61.1, 55.5)
- added R41: 0R, Resistor_SMD:R_0402_1005Metric, F.Cu at (81.3, 73.4)
- added U11: MCP1700x-330xxTT, Package_TO_SOT_SMD:SOT-23, F.Cu at (107.0, 53.2)
- moved C23 2.02 mm to (104.3, 55.1)
- moved U10 1.74 mm to (112.1, 53.6)
- moved C24 1.74 mm to (112.6, 51.1)
- moved R39 1.74 mm to (114.7, 54.1)
- moved U6 1.62 mm to (100.4, 55.2)
- moved R38 1.62 mm to (103.0, 55.6)
- moved R23 1.32 mm to (97.0, 52.1)
- moved R35 1.12 mm to (106.4, 50.2)
- moved Q2 0.30 mm to (67.0, 64.9), turned to 90 degrees
- moved R1 0.14 mm to (82.8, 69.6)
Connections:
- C1 pad 1: +3V3 -> VPP
- C2 pad 2: +5V -> VPP
- C22 pad 2: +3V3 -> VPP
- C23 pad 2: +5V -> +3V3
- C24 pad 2: +5V -> +3V3
- Q2 pad 2: +5V -> Net-(D1-K)
- Q2 pad 3: Net-(D1-K) -> +5V
- Q3 pad 2: +5V -> +3V3
- R1 pad 1: +3V3 -> VPP
- R35 pad 2: +5V -> +3V3
- R38 pad 1: +5V -> +3V3
- R39 pad 1: +5V -> +3V3
- R6 pad 1: +5V -> VPP
- R7 pad 1: +5V -> VPP
- R8 pad 2: +5V -> VPP
- U1 pad 1: +3V3 -> VPP
- U1 pad 17: +5V -> Net-(U1-VBUSM)
- U1 pad 20: +3V3 -> VPP
- U10 pad 5: +5V -> +3V3
- U2 pad 4: +5V -> VPP
- U6 pad 5: +5V -> +3V3
Routing:
- net +5V: track 163.5 -> 121.6 mm, vias 11 -> 7
- net VPP: track 0.00 -> 39.7 mm, vias 0 -> 4
- net GND: track 83.1 -> 93.0 mm, vias 43 -> 48
- net +3V3: track 17.2 -> 26.8 mm
- net Net-(U1-VBUSM): track 0.00 -> 6.38 mm, vias 0 -> 2
- net /Dynamixel-TTL/Dynamixel_dir: track 16.8 -> 20.0 mm
- net Net-(Q2-G): track 7.21 -> 4.48 mm, vias 2 -> 0
- net Net-(J1-Pin_2): track 10.00 -> 12.1 mm
- net Net-(R39-Pad2): track 18.1 -> 19.4 mm
- net /Dynamixel-TTL/Rx: track 7.78 -> 8.91 mm
- net +BATT: track 34.6 -> 35.6 mm
- net Net-(D1-K): track 18.2 -> 19.2 mm
- net /Dynamixel-TTL/Tx: track 8.82 -> 9.77 mm
- net Net-(U1-~{XRSTJ}): track 26.7 -> 25.8 mm
- net Net-(J10-Pad1): track 1.71 -> 2.46 mm
- added copper zone on F.Cu, net +BATT

Commit message: [update] gripette + bulkhead -B1 in production @JLCPCB
Parts:
- removed J4: Dynamixel-3, Connector_JST:JST_EH_B3B-EH-A_1x03_P2.50mm_Vertical
- J5, J9: value Dynamixel-3 -> Feetech; footprint Connector_JST:JST_EH_B3B-EH-A_1x03_P2.50mm_Vertical -> Connector_Molex:Molex_SPOX_5267-03A_1x03_P2.50mm_Vertical
- moved J9 5.46 mm to (81.5, 63.2), turned to 90 degrees
- moved J5 5.02 mm to (75.4, 63.2), turned to 90 degrees
Connections:
- J5 pad 1: GND -> /Dynamixel-TTL over USB/Dyn_data
- J5 pad 3: /Dynamixel-TTL over USB/Dyn_data -> GND
- J9 pad 1: GND -> /Dynamixel-TTL over USB/Dyn_data
- J9 pad 3: /Dynamixel-TTL over USB/Dyn_data -> GND
Routing:
- net VBUS: track 16.6 -> 15.5 mm
- net /Dynamixel-TTL over USB/Dyn_data: track 22.6 -> 21.5 mm
- net GND: track 93.0 -> 94.2 mm
Other:
- board text added: "S + ⏚"
