File: elec_gripette_hub_and_dyn/elec_gripette_hub_and_dyn.kicad_pcb (KiCad board)
At the start: 4 copper layers, 65 x 30 mm, 123 parts, among them J1 pico4, J10 Pogo-pin 4mm, J13 Pogo-pin 4mm, J14 Pogo-pin 4mm, J2 JST EH 2, J3 Pogo-pin 4mm, J5 Feetech, J6 Pogo-pin 4mm, J7 Pogo-pin 2A 4mm, J8 Pogo-pin 2A 4mm, J9 Feetech, Q1 MMBT3906, Q2 SI2312CDS-T1-GE3, Q3 MMBT3906, U1 FE1.1s_24-Pin_WQFN, U10 SN74LVC1G126DBVR, U11 MCP1700x-330xxTT, U2 24C02S, U3 CH343P, U4 SN74LVC1G125DBV, U5 SN74LVC1G126DBVR, U6 SN74LVC1G125DBV, U7 AP63205, U8 LM5050-1, U9 TPS54560BDDA, Y1 12MHz

Commit message: [fix] See Gripette_Slip
Parts:
- removed R19: DNP-0R, Resistor_SMD:R_0603_1608Metric
- removed R20: 0R, Resistor_SMD:R_0603_1608Metric
- added J4: Header 3, Connector_PinHeader_1.27mm:PinHeader_1x03_P1.27mm_Vertical, F.Cu at (87.9, 56.0)
- J3, J6: value Pogo-pin 4mm -> DNP - Pogo-pin 4mm
- moved R28 2.73 mm to (91.6, 59.3)
- moved H2 1.48 mm to (86.1, 51.9)
- moved H3 1.48 mm to (93.6, 50.2)
- moved D11 0.58 mm to (87.9, 58.2), turned to 0 degrees
Connections:
- J5 pad 1: /Dynamixel-TTL over USB/Dyn_data -> GND
- J5 pad 3: GND -> /Dynamixel-TTL over USB/Dyn_data
- J9 pad 1: /Dynamixel-TTL over USB/Dyn_data -> GND
- J9 pad 3: GND -> /Dynamixel-TTL over USB/Dyn_data
Routing:
- net GND: track 94.2 -> 111.6 mm, vias 48 -> 50
- net Net-(C16-Pad1): track 18.4 -> 20.3 mm
- net VBUS: track 15.5 -> 16.9 mm
- net Net-(J4-Pin_3): track 2.49 -> 3.57 mm
- net Net-(J4-Pin_2): track 8.29 -> 7.21 mm
- net Net-(J4-Pin_1): track 2.49 -> 3.42 mm
- net /Dynamixel-TTL over USB/Dyn_data: track 21.5 -> 22.0 mm, vias 0 -> 1
Other:
- board text added: "12V"
- board text added: "7V"
- board text added: "ASE01201-B2"
- board text added: "S"
- board text added: "⏚ +"
- board text removed: "ASE01201-B1"
- board text removed: "S + ⏚"
