File: elec_gripette_hub_and_dyn/dynamixel_3_from_rasp.kicad_sch (KiCad schematic)
At the start: 10 parts

Commit message: [update] SCH + PCB B1-RC1
Parts:
- removed FID1, FID2, FID3: DNP Fiducial, Fiducial:Fiducial_1mm_Mask2mm, symbol Mechanical:Fiducial
- removed H1: PCB01200, symbol Library_Pollen:PCB
- removed H2: Logo HF 2025, Library_Pollen:Logo_HF_2025, symbol Library_Pollen:Logo HF 2025
- removed H3: DNP Logo Pollen 2021, Library_Pollen:Logo_Pollen_2021_sq, symbol Library_Pollen:Logo Pollen 2021
- removed H4, H5, H6, H7: M2,5 x 4mm spacer, LCSC_parts_lib:SMD_BD5.6-D4.1_spacer, symbol Mechanical:MountingHole_Pad
- added C23, C24: 100n, Capacitor_SMD:C_0603_1608Metric, symbol Device:C_Small
- added D12: 5V1, Diode_SMD:D_SOD-323, symbol Device:D_Zener
- added J13, J14: Pogo-pin 4mm, LCSC_parts_lib:CONN-TH_YZ95315064P-01_pogo, symbol Library_Pollen:pogo-pin
- added Q3: MMBT3906, Package_TO_SOT_SMD:SOT-23, symbol Transistor_BJT:MMBT3906
- added R33, R34: 0R, Resistor_SMD:R_0402_1005Metric, symbol Device:R_Small
- added R35, R36, R38, R39: 10k, Resistor_SMD:R_0402_1005Metric, symbol Device:R_Small
- added R37: 20k, Resistor_SMD:R_0402_1005Metric, symbol Device:R_Small
- added R40: 150R, Resistor_SMD:R_0402_1005Metric, symbol Device:R_Small
- added TH2: 100R thermistor, Resistor_SMD:R_0603_1608Metric, symbol Device:Thermistor
- added U10: SN74LVC1G126DBVR, Package_TO_SOT_SMD:SOT-23-5, symbol 74xGxx:74LVC1G126
- added U6: SN74LVC1G125DBV, Package_TO_SOT_SMD:SOT-23-5, symbol 74xGxx:74LVC1G125
Connections:
- net GND: now also C23.1, C24.1, D12.2 (A), R37.1, U10.3 (GND), U6.3 (GND)
- new net: Q3.1 (B), R36.2
- new net: R39.2, R40.1, U10.4, U6.2
- new net: J13.1, R34.1
- new net: J14.1, R33.1
- new net: D12.1 (K), R40.2, TH2.1
- new net +5V: C23.2, C24.2, Q3.2 (E), R35.2, R38.1, R39.1, U10.5 (VCC), U6.5 (VCC)
- new net Dyn_data: TH2.2
- new net Dynamixel_dir: Q3.3 (C), R37.2, U10.1, U6.1
- new net Rx: R34.2, R38.2, U6.4
- new net Tx: R33.2, R35.1, R36.1, U10.2
Other:
- removed sheet Dynamixel-TTL
- removed sheet Dynamixel-TTL over USB
- removed sheet Power
- removed sheet USB hub
- note added: "Rx Rasp IO 15 H. pin 10"
- note added: "Tx Rasp IO 14 H. pin 8"
- note removed: ""elec_hub_and_dyn" is a part of the Grabette/Gripette project, it is a under-HAT for rasp zero 2w with a USB hub and a Dynamixel device."
- note removed: "- SO10x: USB connector + Dynamixel/Feetech @7,4V - OpenArm: USB connector + 24V on XT60"
- note removed: "- la rasp zero 2w fait convertisseur module camera vers usb - on ajoute un converto USB-232 pour aller taper dans les moteurs de gripette - un ajoute un hub pour factoriser tout ce petit monde sur un seul câble - on met un DCDC 24->12 - le tout sur un "under-HAT", sous la rasp, histoire de profiter de la paire diff USB sans utiliser de connecteur (juste des pogo-pins) - universel: ça doit fonctio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"
- note removed: "16/04/2026"
- note removed: "A1"
- note removed: "ASE01201"
- note removed: "B1"
- note removed: "Bulkhead adapter"
- note removed: "Camera"
- note removed: "Check"
- note removed: "Comments"
- note removed: "Date"
- note removed: "Designer"
- note removed: "EB"
- note removed: "Fiducials"
- note removed: "Initial drawing"
- note removed: "Motors"
- note removed: "Raspberry PI"
- note removed: "Release"
- note removed: "SN"
- note removed: "Supplying the motors: - through Vbatt (from the XT60): R28 must be populated - through Dxl: R28 must be removed. Motor communication: - USB (Dynamixel-TTL converter): R15 must be populated - Dynamixel: R15 must be removed."
- note removed: "ToDo: - DXL/Feetech compat (DIP switch + MOS?) - add jumper for accessing uart-dynamixel from rasp-uart"
- note removed: "[fix] Spacers in the BoM [fix] DCDC is now 5A capable [fix] USB pogo-pins position [update] 5V DCDC is on Vbus [update] 4 mm spacers/pogo-pins [added] Test points + access to UART-Dynamixel [added] Hub reset rasp-accessible"
- note removed: "dd/mm/2026"

Commit message: [update] review by Claude. Corrections, RC2
Parts:
- added C25, C26: 1u, Capacitor_SMD:C_0603_1608Metric, symbol Device:C_Small
- added U11: MCP1700x-330xxTT, Package_TO_SOT_SMD:SOT-23, symbol Regulator_Linear:MCP1700x-330xxTT
Connections:
- net +5V: now also C25.2, U11.3 (VI); no longer C23.2, C24.2, Q3.2 (E), R35.2, R38.1, R39.1, U10.5 (VCC), U6.5 (VCC)
- net GND: now also C25.1, C26.1, U11.1 (GND)
- new net +3V3: C23.2, C24.2, C26.2, Q3.2 (E), R35.2, R38.1, R39.1, U10.5 (VCC), U11.2 (VO), U6.5 (VCC)
Other:
- note added: "!! 3V3 !!"
