File: elec_gripette_hub_and_dyn/DCDC.kicad_sch (KiCad schematic)
At the start: 36 parts, among them J2 JST EH 2, J7 Pogo-pin 2A 4mm, J8 Pogo-pin 2A 4mm, Q2 SI2312CDS-T1-GE3, U7 AP63205, U8 LM5050-1, U9 TPS54560BDDA

Commit message: [update] gripette + bulkhead -B1 in production @JLCPCB
Parts:
- U9: FT Rotation Offset (none) -> -90
Changed lines of the file:
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@@
+			)
+		)
+		(property "FT Rotation Offset" "-90"
+			(at 129.54 48.26 0)
+			(effects
+				(font
+					(size 1.27 1.27)
+				)
+				(hide yes)
 			)
 		)
