File: elec_gripette_hub_and_dyn/DCDC.kicad_sch (KiCad schematic)
At the start: 36 parts, among them J2 JST EH 2, J7 Pogo-pin 2A 4mm, J8 Pogo-pin 2A 4mm, Q2 SI2312CDS-T1-GE3, U7 AP63205, U8 LM5050-1, U9 TPS54560BDDA

Commit message: [fix] See Gripette_Slip
Parts:
- removed R19: DNP-0R, Resistor_SMD:R_0603_1608Metric, symbol Device:R_Small
- removed R20: 0R, Resistor_SMD:R_0603_1608Metric, symbol Device:R_Small
- added J4: Header 3, Connector_PinHeader_1.27mm:PinHeader_1x03_P1.27mm_Vertical, symbol Connector_Generic:Conn_01x03
- added JP1: Jumper_2, symbol Library_Pollen:Jumper_2
Connections:
- net at R21.1, R22.2: now also J4.1 (Pin_1)
- net at U9.5 (FB): now also J4.2 (Pin_2)
- net at R16.2, R26.2: now also J4.3 (Pin_3)
Other:
- note removed: "Nota: choose output voltage thanks to 0R. Default is 12V."
- moved on the sheet: R22, R26

Commit message: [update] B2 + B1_bulkhead, now qtty 20 @JLCPCB
Parts:
- J4: FT Rotation Offset (none) -> 90; LCSC Part C2937625 -> C7470079
Changed lines of the file:
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@@
 			)
 		)
-		(property "LCSC Part" "C2937625"
+		(property "LCSC Part" "C7470079"
 			(at 209.55 60.96 0)
 			(effects
+				(font
+					(size 1.27 1.27)
+				)
+				(hide yes)
+			)
+		)
+		(property "FT Rotation Offset" "90"
+			(at 209.55 60.96 0)
+			(effects

Commit message: [added] BoMs
Parts:
- J4: FT Rotation Offset 90 -> (none); LCSC Part C7470079 -> C2937625
Changed lines of the file:
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@@
 			)
 		)
-		(property "LCSC Part" "C7470079"
+		(property "LCSC Part" "C2937625"
 			(at 209.55 60.96 0)
 			(effects
-				(font
-					(size 1.27 1.27)
-				)
-				(hide yes)
-			)
-		)
-		(property "FT Rotation Offset" "90"
-			(at 209.55 60.96 0)
-			(effects
