File: elec_gripette_hub_and_dyn/usb_hub.kicad_sch (KiCad schematic)
At the start: 32 parts, among them J1 pico4, J10 Pogo-pin 4mm, J3 Pogo-pin 4mm, J6 Pogo-pin 4mm, U1 FE1.1s_24-Pin_WQFN, U2 24C02S, Y1 12MHz

Commit message: [update] gripette + bulkhead -B1 in production @JLCPCB
Parts:
- D5: FT Rotation Offset (none) -> 180
Changed lines of the file:
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@@
 			)
 		)
-		(property "FT Rotation Offset" ""
+		(property "FT Rotation Offset" "180"
 			(at 252.73 157.48 90)
 			(effects
