File: elec_gripette_hub_and_dyn/usb_hub.kicad_sch (KiCad schematic)
At the start: 32 parts, among them J1 pico4, J10 Pogo-pin 4mm, J3 Pogo-pin 4mm, J6 Pogo-pin 4mm, U1 FE1.1s_24-Pin_WQFN, U2 24C02S, Y1 12MHz

Commit message: [fix] See Gripette_Slip
Parts:
- J3, J6: value Pogo-pin 4mm -> DNP - Pogo-pin 4mm; now not fitted
Changed lines of the file:
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@@
 		(in_bom yes)
 		(on_board yes)
-		(dnp no)
+		(dnp yes)
 		(property "Reference" "J6"
 			(at 268.224 82.296 90)
@@
 			)
 		)
-		(property "Value" "Pogo-pin 4mm"
+		(property "Value" "DNP - Pogo-pin 4mm"
 			(at 261.62 84.8532 90)
 			(effects
@@
 		(in_bom yes)
 		(on_board yes)
-		(dnp no)
+		(dnp yes)
 		(property "Reference" "J3"
 			(at 257.81 82.3132 90)
@@
 			)
 		)
-		(property "Value" "Pogo-pin 4mm"
+		(property "Value" "DNP - Pogo-pin 4mm"
 			(at 257.81 84.8532 90)
 			(effects
