File: elec_gripette_hub_and_dyn/dynamixel_3.kicad_sch (KiCad schematic)
At the start: 26 parts, among them J5 Feetech, J9 Feetech, Q1 MMBT3906, U3 CH343P, U4 SN74LVC1G125DBV, U5 SN74LVC1G126DBVR

Commit message: [fix] See Gripette_Slip
Connections:
- net Dyn_data: now also J5.3 (Pin_3), J9.3 (Pin_3); no longer J5.1 (Pin_1), J9.1 (Pin_1)
- net GND: now also J5.1 (Pin_1), J9.1 (Pin_1); no longer J5.3 (Pin_3), J9.3 (Pin_3)
Changed lines of the file:
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@@
 		(lib_id "Connector_Generic:Conn_01x03")
 		(at 334.01 191.77 0)
+		(mirror x)
 		(unit 1)
 		(exclude_from_sim no)
@@
 		)
 		(property "Value" "Feetech"
-			(at 337.82 194.31 0)
+			(at 337.82 189.23 0)
 			(effects
 				(font
@@
 		(lib_id "Connector_Generic:Conn_01x03")
 		(at 334.01 176.53 0)
+		(mirror x)
 		(unit 1)
 		(exclude_from_sim no)
@@
 		)
 		(property "Value" "Feetech"
-			(at 337.82 179.07 0)
+			(at 337.82 173.99 0)
 			(effects
 				(font
