File: elec_gripette_hub_and_dyn/elec_gripette_hub_and_dyn.kicad_sch (KiCad schematic)
At the start: 10 parts

Commit message: [fix] See Gripette_Slip
Other:
- note added: "07/07/2026"
- note added: "[fix] DNP USB-pogo pins [fix] Motor conn. -> Feetech [update] Motor voltage selection"
- note removed: "- SO10x: USB connector + Dynamixel/Feetech @7,4V - OpenArm: USB connector + 24V on XT60"
- note removed: "- la rasp zero 2w fait convertisseur module camera vers usb - on ajoute un converto USB-232 pour aller taper dans les moteurs de gripette - un ajoute un hub pour factoriser tout ce petit monde sur un seul câble - on met un DCDC 24->12 - le tout sur un "under-HAT", sous la rasp, histoire de profiter de la paire diff USB sans utiliser de connecteur (juste des pogo-pins) - universel: ça doit fonctio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"
- note removed: "29/06/2026"
- note removed: "TODO: - nopop pogo - easier motor voltage selection - fix motor connector to Feetech"

Commit message: [update] ToDo for SO100
Other:
- note added: "ToDo: - still the USB does not operate (pogo-pins? rasp-gadget-mode?) - for using only the dynamixel/feetech, one need to remove R28, but then it is required to inject Vbus into Vbat: add an extra 0R for that."
Changed lines of the file:
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@@
+		)
+	)
+	(text "ToDo:\n - still the USB does not operate (pogo-pins? rasp-gadget-mode?)\n - for using only the dynamixel/feetech, one need to remove R28, \n   but then it is required to inject Vbus into Vbat: add an extra\n   0R for that."
+		(exclude_from_sim no)
+		(at 54.61 92.71 0)
+		(effects
+			(font
+				(size 2.0066 2.0066)
+			)
+			(justify left bottom)
 		)
 	)
