File: elec_gripette_hub_and_dyn/Bulkhead_Adapters/elec_bulkhead_XT30_USB-C/elec_bulkhead_XT60_USB-C.kicad_sch (KiCad schematic)
At the start: 20 parts, among them J1 USB-C Rec. Vert., J2 JST EH 2, J3 XT30, J4 pico4, J5 Dynamixel-3, J6 USB_C_Receptacle, J8 USB3_A, J9 Dynamixel-3

Commit message: [update] Gripette Bulkhead DNP Dyn c.
Parts:
- J5, J9: value Dynamixel-3 -> DNP - Dynamixel-3; now not fitted
Other:
- note added: "B1"
- note added: "ToDo: - Change Dynamixel connectors for Feetech?"

Commit message: [fix] Bulkhead -> B2 because of a USB-C/3 extra locator pin
Other:
- note added: "16/07/2026"
- note added: "B2"
- note added: "[fix] USB-C/3 extra monting pin"
Changed lines of the file:
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@@
+		)
+	)
+	(text "B2"
+		(exclude_from_sim no)
+		(at 140.97 56.642 0)
+		(effects
+			(font
+				(size 2.0066 2.0066)
+			)
+			(justify left bottom)
 		)
 	)
@@
 		)
 	)
+	(text "SN"
+		(exclude_from_sim no)
+		(at 200.66 56.642 0)
+		(effects
+			(font
+				(size 2.0066 2.0066)
+			)
+			(justify left bottom)
+		)
+	)
 	(text "B1"
 		(exclude_from_sim no)
@@
 		)
 	)
+	(text "EB"
+		(exclude_from_sim no)
+		(at 185.42 56.642 0)
+		(effects
+			(font
+				(size 2.0066 2.0066)
+			)
+			(justify left bottom)
+		)
+	)
 	(text "\"elec_bulkhead_XT30_USB-C\" is a dedicated to Gripette project."
 		(exclude_from_sim no)
@@
 		(exclude_from_sim no)
 		(at 184.15 35.56 0)
+		(effects
+			(font
+				(size 2.0066 2.0066)
+			)
+			(justify left bottom)
+		)
+	)
+	(text "16/07/2026"
+		(exclude_from_sim no)
+		(at 161.29 56.642 0)
 		(effects
 			(font
@@
 		)
 	)
+	(text "[fix] USB-C/3 extra monting pin"
+		(exclude_from_sim no)
+		(at 214.884 56.388 0)
+		(effects
+			(font
+				(size 2.0066 2.0066)
+			)
+			(justify left bottom)
+		)
+	)
 	(text "SN"
 		(exclude_from_sim no)
@@
 			(type default)
 		)
+	)
+	(polyline
+		(pts
+			(xy 140.97 52.07) (xy 275.59 52.07)
+		)
+		(stroke
+			(width 0)
+			(type default)
+		)
