File: elec_DCDC/elec_DCDC.kicad_pcb (KiCad board)
At the start: 2 copper layers, 36 x 20 mm, 29 parts, among them J1 XT30, J2 Dynamixel-3, U1 MP2338

Commit message: [fix] See Gripette_Slip
Routing:
- net (no net): track 24.3 -> 0.00 mm
- net GND: track 1.76 -> 0.00 mm
Changed lines of the file:
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@@
 		)
-	)
-	(segment
-		(start 128.422501 53.065001)
-		(end 128.422501 51.545001)
-		(width 0.5)
-		(layer "B.Cu")
-		(net 0)
-	)
-	(segment
-		(start 128.547501 53.190001)
-		(end 128.422501 53.065001)
-		(width 0.5)
-		(layer "B.Cu")
-		(net 0)
-	)
-	(segment
-		(start 130.597501 51.040001)
-		(end 130.597501 50.240001)
-		(width 0.5)
-		(layer "B.Cu")
-		(net 0)
-	)
-	(segment
-		(start 133.372501 49.005001)
-		(end 132.132501 49.005001)
-		(width 0.3)
-		(layer "B.Cu")
-		(net 0)
-	)
-	(segment
-		(start 130.597501 50.240001)
-		(end 130.597501 46.140001)
-		(width 0.5)
-		(layer "B.Cu")
-		(net 0)
-	)
-	(segment
-		(start 134.397501 46.440001)
-		(end 132.997501 46.440001)
-		(width 0.3)
-		(layer "B.Cu")
-		(net 0)
-	)
-	(segment
-		(start 130.562501 50.275001)
-		(end 130.597501 50.240001)
-		(width 0.5)
-		(layer "B.Cu")
-		(net 0)
-	)
-	(segment
-		(start 128.422501 51.545001)
-		(end 130.092501 51.545001)
-		(width 0.5)
-		(layer "B.Cu")
-		(net 0)
-	)
-	(segment
-		(start 133.372501 50.275001)
-		(end 134.562501 50.275001)
-		(width 0.3)
-		(layer "B.Cu")
-		(net 0)
-	)
-	(segment
-		(start 132.132501 49.005001)
-		(end 131.497501 49.640001)
-		(width 0.3)
-		(layer "B.Cu")
-		(net 0)
-	)
-	(segment
-		(start 128.422501 50.275001)
-		(end 130.562501 50.275001)
-		(width 0.5)
-		(layer "B.Cu")
-		(net 0)
-	)
-	(segment
-		(start 135.097501 47.140001)
-		(end 134.397501 46.440001)
-		(width 0.3)
-		(layer "B.Cu")
-		(net 0)
-	)
-	(segment
-		(start 130.092501 51.545001)
-		(end 130.597501 51.040001)
-		(width 0.5)
-		(layer "B.Cu")
-		(net 0)
-	)
-	(segment
-		(start 131.497501 49.640001)
-		(end 131.497501 53.240001)
-		(width 0.3)
-		(layer "B.Cu")
-		(net 0)
-	)
-	(segment
-		(start 128.547501 53.240001)
-		(end 128.547501 53.190001)
-		(width 0.5)
-		(layer "B.Cu")
-		(net 0)
-	)
-	(segment
-		(start 135.097501 49.740001)
-		(end 135.097501 47.140001)
-		(width 0.3)
-		(layer "B.Cu")
-		(net 0)
-	)
-	(segment
-		(start 130.597501 46.140001)
-		(end 130.877501 45.860001)
-		(width 0.5)
-		(layer "B.Cu")
-		(net 0)
-	)
-	(segment
-		(start 134.562501 50.275001)
-		(end 135.097501 49.740001)
-		(width 0.3)
-		(layer "B.Cu")
-		(net 0)
-	)
-	(segment
-		(start 128.397501 47.710001)
-		(end 128.422501 47.735001)
-		(width 0.5)
-		(layer "B.Cu")
-		(net 1)
-	)
-	(segment
-		(start 128.397501 46.540001)
-		(end 128.397501 47.710001)
-		(width 0.5)
-		(layer "B.Cu")
-		(net 1)
-	)
-	(segment
-		(start 132.897501 51.740001)
-		(end 133.177501 51.740001)
-		(width 0.5)
-		(layer "B.Cu")
-		(net 1)
-	)
-	(segment
-		(start 133.177501 51.740001)
-		(end 133.372501 51.545001)
-		(width 0.5)
-		(layer "B.Cu")
-		(net 1)
 	)
 	(group ""
