File: elec_DCDC/elec_DCDC.kicad_sch (KiCad schematic)
At the start: 30 parts, among them J1 XT30, J2 Dynamixel-3, U1 MP2338

Commit message: [fix] See Gripette_Slip
Other:
- note added: "Todo: - ideal diode to avoid reverse supplying?"
Changed lines of the file:
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@@
+		)
+	)
+	(text "Todo:\n - ideal diode to avoid reverse supplying?"
+		(exclude_from_sim no)
+		(at 106.68 82.55 0)
+		(effects
+			(font
+				(size 2.0066 2.0066)
+			)
+			(justify left bottom)
 		)
 	)
