File: elec_HMI/elec_HMI.kicad_sch (KiCad schematic)
At the start: 17 parts, among them J1 JST SH, Q1 MMBT3906, SW1 SW_SPST

Commit message: [added] Production files
Other:
- note added: "17/03/2026"
- note removed: "dd/mm/2026"
