File: elec_IMU/elec_IMU.kicad_sch (KiCad schematic)
At the start: 22 parts, among them J1 JST SH, J2 JST SH, U1 BMI088

Commit message: [added] Production files
Other:
- note added: "12/03/2026"
- note removed: "dd/mm/2026"
